File: PCB_design/Lab2.kicad_pcb (KiCad board)
At the start: 2 copper layers, 39.4 x 38.1 mm, 12 parts, among them J1 Conn_01x02_Pin, U1 NE555D

Commit message: Lab2
Other:
- board size 39.4 x 38.1 mm -> 51 x 48 mm
Changed lines of the file:
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@@
   (gr_rect (start 52.07 50.8) (end 57.15 55.88)
+    (stroke (width 0.1) (type default)) (fill none) (layer "Edge.Cuts"))
+  (gr_rect (start 12 12) (end 63 60)
     (stroke (width 0.1) (type default)) (fill none) (layer "Edge.Cuts"))
   (gr_rect (start 17.78 17.78) (end 22.86 22.86)
